Commit message: Fix robot mass and caster wheel position

File: alphabot_world/robots/alphabot2.xacro (robot description, xacro)
@@ -76,5 +76,5 @@
     </collision>
     <visual name="caster_front_visual">
-      <origin rpy="0 0 0" xyz="0.05 0 -0.0335"/>
+      <origin rpy="0 0 0" xyz="0.05 0 -0.0325"/>
       <geometry>
         <sphere radius="0.005"/>
@@ -85,5 +85,5 @@
     <!-- caster back collision and visual -->
     <collision name="caster_back_collision">
-      <origin rpy="0 0 0" xyz="-0.05 0 -0.0335"/>
+      <origin rpy="0 0 0" xyz="-0.05 0 -0.0325"/>
       <geometry>
         <sphere radius="0.005"/>
@@ -113,5 +113,5 @@
   <link name="link_right_wheel">
     <inertial>
-      <mass value="0.025"/>
+      <mass value="0.045"/>
       <origin rpy="0 1.5707 1.5707" xyz="0 0 0"/>
       <inertia ixx="0.00052666666" ixy="0" ixz="0" iyy="0.00052666666" iyz="0" izz="0.001"/>
@@ -145,5 +145,5 @@
   <link name="link_left_wheel">
     <inertial>
-      <mass value="0.025"/>
+      <mass value="0.045"/>
       <origin rpy="0 1.5707 1.5707" xyz="0 0 0"/>
       <inertia ixx="0.00052666666" ixy="0" ixz="0" iyy="0.00052666666" iyz="0" izz="0.001"/>
