Commit message: Fix Rviz and Launch files

File: alphabot2_world/robots/wheel_macro.xacro (robot description, xacro)
@@ -29,5 +29,5 @@
     <joint name="${name}" type="continuous">
       <origin rpy="0 0 0" xyz="${origin_xyz}"/>
-      <child link="${name}"/>
+      <child link="${child}"/>
       <parent link="link_chassis"/>
       <axis rpy="0 0 0" xyz="0 1 0"/>
