Commit message: Change Urdf visual file

File: alphabot2_world/robots/alphabot2.xacro (robot description, xacro)
@@ -51,7 +51,7 @@
     </collision>
     <visual>
-      <origin rpy="0 0 0" xyz="0 0 0"/>
+      <origin rpy="0 0 0" xyz="0 0 -0.0225"/>
       <geometry>
-        <cylinder radius="0.055" length="0.045"/>
+        <mesh filename="package://alphabot2_world/meshes/chassis.stl" />
       </geometry>
       <material name="blue"/>
@@ -60,5 +60,5 @@
     <!-- caster front collision and visual -->
     <collision name="caster_front_collision">
-      <origin rpy="0 0 0" xyz="0.05 0 -0.0335"/>
+      <origin rpy="0 0 0" xyz="0.05 0 -0.03"/>
       <geometry>
         <sphere radius="0.005"/>
@@ -76,5 +76,5 @@
     </collision>
     <visual name="caster_front_visual">
-      <origin rpy="0 0 0" xyz="0.05 0 -0.0325"/>
+      <origin rpy="0 0 0" xyz="0.05 0 -0.03"/>
       <geometry>
         <sphere radius="0.005"/>
@@ -85,5 +85,5 @@
     <!-- caster back collision and visual -->
     <collision name="caster_back_collision">
-      <origin rpy="0 0 0" xyz="-0.05 0 -0.0325"/>
+      <origin rpy="0 0 0" xyz="-0.05 0 -0.03"/>
       <geometry>
         <sphere radius="0.005"/>
@@ -101,5 +101,5 @@
     </collision>
     <visual name="caster_back_visual">
-      <origin rpy="0 0 0" xyz="-0.05 0 -0.0335"/>
+      <origin rpy="0 0 0" xyz="-0.05 0 -0.03"/>
       <geometry>
         <sphere radius="0.005"/>

Commit message: Add macro files

File: alphabot2_world/robots/alphabot2.xacro (robot description, xacro)
@@ -1,37 +1,8 @@
 <?xml version="1.0" ?>
 <robot name="alphabot2" xmlns:xacro="https://www.ros.org/wiki/xacro" >
-  <material name="black">
-    <color rgba="0.0 0.0 0.0 1.0"/>
-  </material>
-  <material name="blue">
-    <color rgba="0.203125 0.23828125 0.28515625 1.0"/>
-  </material>
-  <material name="green">
-    <color rgba="0.0 0.8 0.0 1.0"/>
-  </material>
-  <material name="grey">
-    <color rgba="0.2 0.2 0.2 1.0"/>
-  </material>
-  <material name="orange">
-    <color rgba="1.0 0.423529411765 0.0392156862745 1.0"/>
-  </material>
-  <material name="brown">
-    <color rgba="0.870588235294 0.811764705882 0.764705882353 1.0"/>
-  </material>
-  <material name="red">
-    <color rgba="0.80078125 0.12890625 0.1328125 1.0"/>
-  </material>
-  <material name="white">
-    <color rgba="1.0 1.0 1.0 1.0"/>
-  </material>
-  <gazebo reference="link_chassis">
-    <material>Gazebo/Blue</material>
-  </gazebo>
-  <gazebo reference="link_left_wheel">
-    <material>Gazebo/Black</material>
-  </gazebo>
-  <gazebo reference="link_right_wheel">
-    <material>Gazebo/Black</material>
-  </gazebo>
+  <xacro:include filename="$(find alphabot2_world)/robots/materials.xacro" />
+  <xacro:include filename="$(find alphabot2_world)/robots/gazebo.xacro" />
+  <xacro:include filename="$(find alphabot2_world)/robots/wheel_macro.xacro" />
+  <xacro:include filename="$(find alphabot2_world)/robots/caster_macro.xacro" />
   <!-- chassis -->
   <link name="link_chassis">
@@ -58,135 +29,23 @@
     </visual>
     <!-- end of chassis collision and visual -->
-    <!-- caster front collision and visual -->
-    <collision name="caster_front_collision">
-      <origin rpy="0 0 0" xyz="0.05 0 -0.03"/>
-      <geometry>
-        <sphere radius="0.005"/>
-      </geometry>
-      <surface>
-        <friction>
-          <ode>
-            <mu>0</mu>
-            <mu2>0</mu2>
-            <slip1>1.0</slip1>
-            <slip2>1.0</slip2>
-          </ode>
-        </friction>
-      </surface>
-    </collision>
-    <visual name="caster_front_visual">
-      <origin rpy="0 0 0" xyz="0.05 0 -0.03"/>
-      <geometry>
-        <sphere radius="0.005"/>
-      </geometry>
-      <material name="white"/>
-    </visual>
-    <!-- end of caster front collision and visual -->
-    <!-- caster back collision and visual -->
-    <collision name="caster_back_collision">
-      <origin rpy="0 0 0" xyz="-0.05 0 -0.03"/>
-      <geometry>
-        <sphere radius="0.005"/>
-      </geometry>
-      <surface>
-        <friction>
-          <ode>
-            <mu>0</mu>
-            <mu2>0</mu2>
-            <slip1>1.0</slip1>
-            <slip2>1.0</slip2>
-          </ode>
-        </friction>
-      </surface>
-    </collision>
-    <visual name="caster_back_visual">
-      <origin rpy="0 0 0" xyz="-0.05 0 -0.03"/>
-      <geometry>
-        <sphere radius="0.005"/>
-      </geometry>
-      <material name="white"/>
-    </visual>
-    <!-- end of caster back collision and visual -->
+    <!-- caster front -->
+    <xacro:caster name="caster_front"  origin_xyz="0.05 0 -0.03"  />
+    <!-- end of caster front -->
+    <!-- caster back -->
+    <xacro:caster name="caster_back"  origin_xyz="-0.05 0 -0.03"  />
+    <!-- end of caster back -->
   </link>
   <!-- end of chassis -->
   <!-- right wheel -->
-  <link name="link_right_wheel">
-    <inertial>
-      <mass value="0.045"/>
-      <origin rpy="0 1.5707 1.5707" xyz="0 0 0"/>
-      <inertia ixx="0.00052666666" ixy="0" ixz="0" iyy="0.00052666666" iyz="0" izz="0.001"/>
-    </inertial>
-    <collision name="link_right_wheel_collision">
-      <origin rpy="0 1.5707 1.5707" xyz="0 0 0" />
-      <geometry>
-        <cylinder length="0.017" radius="0.021"/>
-      </geometry>
-    </collision>
-    <visual name="link_right_wheel_visual">
-      <origin rpy="0 1.5707 1.5707" xyz="0 0 0"/>
-      <geometry>
-        <cylinder length="0.017" radius="0.021"/>
-      </geometry>
-      <material name="black"/>
-    </visual>
-  </link>
+  <xacro:link_wheel name="link_right_wheel" />
   <!-- end of right wheel -->
   <!-- joint for right wheel -->
-  <joint name="joint_right_wheel" type="continuous">
-    <origin rpy="0 0 0" xyz="0 0.046 -0.016"/>
-    <child link="link_right_wheel" />
-    <parent link="link_chassis"/>
-    <axis rpy="0 0 0" xyz="0 1 0"/>
-    <limit effort="10000" velocity="1000"/>
-    <joint_properties damping="1.0" friction="1.0" />
-  </joint>
+  <xacro:joint_wheel name="joint_right_wheel"  child="link_right_wheel"  origin_xyz="0 0.046 -0.016"  />
   <!-- end of joint for right wheel -->
   <!-- left wheel -->
-  <link name="link_left_wheel">
-    <inertial>
-      <mass value="0.045"/>
-      <origin rpy="0 1.5707 1.5707" xyz="0 0 0"/>
-      <inertia ixx="0.00052666666" ixy="0" ixz="0" iyy="0.00052666666" iyz="0" izz="0.001"/>
-    </inertial>
-    <collision name="link_left_wheel_collision">
-      <origin rpy="0 1.5707 1.5707" xyz="0 0 0" />
-      <geometry>
-        <cylinder length="0.017" radius="0.021"/>
-      </geometry>
-    </collision>
-    <visual name="link_left_wheel_visual">
-      <origin rpy="0 1.5707 1.5707" xyz="0 0 0"/>
-      <geometry>
-        <cylinder length="0.017" radius="0.021"/>
-      </geometry>
-      <material name="black"/>
-    </visual>
-  </link>
+  <xacro:link_wheel name="link_left_wheel" />
   <!-- end of left wheel -->
   <!-- joint for left wheel -->
-  <joint name="joint_left_wheel" type="continuous">
-    <origin rpy="0 0 0" xyz="0 -0.046 -0.016"/>
-    <child link="link_left_wheel" />
-    <parent link="link_chassis"/>
-    <axis rpy="0 0 0" xyz="0 1 0"/>
-    <limit effort="10000" velocity="1000"/>
-    <joint_properties damping="1.0" friction="1.0" />
-  </joint>
+  <xacro:joint_wheel name="joint_left_wheel"   child="link_left_wheel"   origin_xyz="0 -0.046 -0.016"  />
   <!-- end of joint for left wheel -->
-  <!-- Diferential Control -->
-  <gazebo>
-    <plugin filename="libgazebo_ros_diff_drive.so" name="differential_drive_controller">
-      <alwaysOn>true</alwaysOn>
-      <updateRate>20</updateRate>
-      <leftJoint>joint_left_wheel</leftJoint>
-      <rightJoint>joint_right_wheel</rightJoint>
-      <wheelSeparation>0.4</wheelSeparation>
-      <wheelDiameter>0.2</wheelDiameter>
-      <torque>0.1</torque>
-      <commandTopic>cmd_vel</commandTopic>
-      <odometryTopic>odom</odometryTopic>
-      <odometryFrame>odom</odometryFrame>
-      <robotBaseFrame>link_chassis</robotBaseFrame>
-    </plugin>
-  </gazebo>
 </robot>

Commit message: Add camera link

File: alphabot2_world/robots/alphabot2.xacro (robot description, xacro)
@@ -49,3 +49,119 @@
   <xacro:joint_wheel name="joint_left_wheel"   child="link_left_wheel"   origin_xyz="0 -0.046 -0.016"  />
   <!-- end of joint for left wheel -->
+  <link name="lower_camera_link">
+  <inertial>
+      <mass value="0.0225"/>
+      <origin rpy="0 0 0" xyz="0 0 0"/>
+      <inertia ixx="0.0000058388" ixy="0" ixz="0" iyy="0.0000063638" iyz="0" izz="0.0000046088"/>
+  </inertial>
+  <collision name="lower_camera_collision">
+      <origin rpy="0 0 0" xyz="0 0 0" />
+      <geometry>
+        <box size="0.037 0.033 0.045"/>
+      </geometry>
+  </collision>
+  <visual name="lower_camera_visual">
+      <origin rpy="0 0 0" xyz="0 0 0"/>
+      <geometry>
+        <box size="0.037 0.033 0.045"/>
+      </geometry>
+      <material name="red"/>
+  </visual>
+  </link>
+   <joint name="joint_lower_camera_link" type="continuous">
+    <origin rpy="0 0 0" xyz="0 0 0.045"/>
+    <child link="lower_camera_link" />
+    <parent link="link_chassis"/>
+    <axis rpy="0 0 0" xyz="0 0 1"/>
+    <limit effort="10000" velocity="1000" lower="-1.57" upper="1.57"/>
+    <joint_properties damping="1.0" friction="1.0" />
+  </joint>
+  <!--TODO: plugin link da câmara de baixo-->
+  <link name="upper_camera_link">
+  <inertial>
+      <mass value="0.0225"/>
+      <origin rpy="0 0 0" xyz="0 0 0"/>
+      <inertia ixx="0" ixy="0" ixz="0" iyy="0.000006" iyz="0" izz="0.000005"/>
+  </inertial>
+  <collision name="upper_camera_collision">
+      <origin rpy="0 0 0" xyz="0 0 0" />
+      <geometry>
+        <mesh filename="package://alphabot2_world/meshes/chassis.stl" />
+      </geometry>
+  </collision>
+  <visual name="lower_camera_link_visual">
+      <origin rpy="0 0 0" xyz="0 0 0"/>
+      <geometry>
+        <mesh filename="package://alphabot2_world/meshes/camera.stl" />
+      </geometry>
+      <material name="orange"/>
+  </visual>
+  </link>
+   <joint name="joint_upper_camera_link" type="continuous">
+    <origin rpy="0 0 0" xyz="0 0 0.045"/>
+    <child link="upper_camera_link" />
+    <parent link="lower_camera_link"/>
+    <axis rpy="0 0 0" xyz="0 0 1"/>
+    <limit effort="10000" velocity="1000" lower="-1.57" upper="1.57"/>
+    <joint_properties damping="1.0" friction="1.0" />
+  </joint>
+  <!-- camera -->
+  <gazebo reference="camera_link">
+    <sensor type="camera" name="camera">
+      <update_rate>30.0</update_rate>
+      <camera name="head">
+      <save enabled="true">
+              <path>/tmp/</path>
+            </save>
+        <horizontal_fov>1.08504</horizontal_fov>
+        <image>
+          <width>2552</width>
+          <height>1944</height>
+          <!--format>R8G8B8</format-->
+        </image>
+        <clip>
+          <near>0.01</near>
+          <far>1000</far>
+        </clip>
+        <noise>
+          <type>gaussian</type>
+          <!-- Noise is sampled independently per pixel on each frame.
+               That pixel's noise value is added to each of its color
+               channels, which at that point lie in the range [0,1]. -->
+          <mean>0.0</mean>
+          <stddev>0.007</stddev>
+        </noise>
+      </camera>
+      <plugin name="camera_controller" filename="libgazebo_ros_camera.so">
+        <alwaysOn>true</alwaysOn>
+        <updateRate>0.0</updateRate>
+        <cameraName>alphabot2/camera</cameraName>
+        <imageTopicName>image_raw</imageTopicName>
+        <cameraInfoTopicName>camera_info</cameraInfoTopicName>
+        <frameName>camera_link</frameName>
+        <hackBaseline>0.07</hackBaseline>
+        <distortionK1>0.0</distortionK1>
+        <distortionK2>0.0</distortionK2>
+        <distortionK3>0.0</distortionK3>
+        <distortionT1>0.0</distortionT1>
+        <distortionT2>0.0</distortionT2>
+      </plugin>
+    </sensor>
+  </gazebo>
+  <!-- Diferential Control -->
+  <gazebo>
+    <plugin filename="libgazebo_ros_diff_drive.so" name="differential_drive_controller">
+      <alwaysOn>true</alwaysOn>
+      <updateRate>20</updateRate>
+      <leftJoint>joint_left_wheel</leftJoint>
+      <rightJoint>joint_right_wheel</rightJoint>
+      <wheelSeparation>0.4</wheelSeparation>
+      <wheelDiameter>0.2</wheelDiameter>
+      <torque>0.1</torque>
+      <commandTopic>cmd_vel</commandTopic>
+      <odometryTopic>odom</odometryTopic>
+      <odometryFrame>odom</odometryFrame>
+      <robotBaseFrame>link_chassis</robotBaseFrame>
+    </plugin>
+  </gazebo>
 </robot>

Commit message: 'Fix camera'

File: alphabot2_world/robots/alphabot2.xacro (robot description, xacro)
@@ -77,46 +77,50 @@
     <joint_properties damping="1.0" friction="1.0" />
   </joint>
-  <!--TODO: plugin link da câmara de baixo-->
+  <!--TODO: plugin link da camara de baixo-->
   <link name="upper_camera_link">
+    <origin rpy="0 0 0" xyz="0 0 0"/>
   <inertial>
       <mass value="0.0225"/>
-      <origin rpy="0 0 0" xyz="0 0 0"/>
+      <origin rpy="0 ${3.14/2} 0" xyz="0 0 0 "/>
       <inertia ixx="0" ixy="0" ixz="0" iyy="0.000006" iyz="0" izz="0.000005"/>
   </inertial>
   <collision name="upper_camera_collision">
-      <origin rpy="0 0 0" xyz="0 0 0" />
+      <origin rpy="0 ${3.14/2} 0" xyz="0 0 0" />
       <geometry>
         <mesh filename="package://alphabot2_world/meshes/chassis.stl" />
       </geometry>
   </collision>
-  <visual name="lower_camera_link_visual">
-      <origin rpy="0 0 0" xyz="0 0 0"/>
+  <visual name="upper_camera_visual">
+      <origin rpy="0 ${3.14/2} 0" xyz="0 0 0"/>
       <geometry>
         <mesh filename="package://alphabot2_world/meshes/camera.stl" />
       </geometry>
-      <material name="orange"/>
+      <material name="blue"/>
   </visual>
   </link>
    <joint name="joint_upper_camera_link" type="continuous">
-    <origin rpy="0 0 0" xyz="0 0 0.045"/>
+    <origin rpy="0 ${-3.14/2} 0" xyz="0 0 0.045"/>
     <child link="upper_camera_link" />
     <parent link="lower_camera_link"/>
-    <axis rpy="0 0 0" xyz="0 0 1"/>
+    <axis rpy="0 0 0" xyz="0 1 0"/>
     <limit effort="10000" velocity="1000" lower="-1.57" upper="1.57"/>
     <joint_properties damping="1.0" friction="1.0" />
   </joint>
   <!-- camera -->
-  <gazebo reference="camera_link">
-    <sensor type="camera" name="camera">
+  <gazebo reference="upper_camera_link">
+    <sensor name="alphabot2_camera" type="camera" >
+      <visualize>1</visualize>
+      <always_on>1</always_on>
       <update_rate>30.0</update_rate>
-      <camera name="head">
-      <save enabled="true">
-              <path>/tmp/</path>
-            </save>
+      <camera name="alphabot2_camera">
+      <origin rpy="0 ${3.14/2} 0" xyz="0.015 0 0.045"/>
+        <save enabled="true">
+          <path>/tmp/</path>
+        </save>
         <horizontal_fov>1.08504</horizontal_fov>
         <image>
-          <width>2552</width>
-          <height>1944</height>
-          <!--format>R8G8B8</format-->
+          <width>160</width>
+          <height>120</height>
+          <format>R8G8B8</format>
         </image>
         <clip>
@@ -135,6 +139,6 @@
       <plugin name="camera_controller" filename="libgazebo_ros_camera.so">
         <alwaysOn>true</alwaysOn>
-        <updateRate>0.0</updateRate>
-        <cameraName>alphabot2/camera</cameraName>
+        <updateRate>30.0</updateRate>
+        <cameraName>alphabot2_camera/</cameraName>
         <imageTopicName>image_raw</imageTopicName>
         <cameraInfoTopicName>camera_info</cameraInfoTopicName>
@@ -149,19 +153,3 @@
     </sensor>
   </gazebo>
-  <!-- Diferential Control -->
-  <gazebo>
-    <plugin filename="libgazebo_ros_diff_drive.so" name="differential_drive_controller">
-      <alwaysOn>true</alwaysOn>
-      <updateRate>20</updateRate>
-      <leftJoint>joint_left_wheel</leftJoint>
-      <rightJoint>joint_right_wheel</rightJoint>
-      <wheelSeparation>0.4</wheelSeparation>
-      <wheelDiameter>0.2</wheelDiameter>
-      <torque>0.1</torque>
-      <commandTopic>cmd_vel</commandTopic>
-      <odometryTopic>odom</odometryTopic>
-      <odometryFrame>odom</odometryFrame>
-      <robotBaseFrame>link_chassis</robotBaseFrame>
-    </plugin>
-  </gazebo>
 </robot>
