Commit message: sensors added to xacro and publishing values

File: alphabot2_world/robots/alphabot2.xacro (robot description, xacro)
@@ -49,5 +49,5 @@
   <xacro:joint_wheel name="joint_left_wheel"   child="link_left_wheel"   origin_xyz="0 -0.046 -0.016"  />
   <!-- end of joint for left wheel -->
-  <link name="lower_camera_link">
+  <!--<link name="lower_camera_link">
   <inertial>
       <mass value="0.0225"/>
@@ -76,7 +76,7 @@
     <limit effort="10000" velocity="1000" lower="-1.57" upper="1.57"/>
     <joint_properties damping="1.0" friction="1.0" />
-  </joint>
+  </joint>-->
   <!--TODO: plugin link da camara de baixo-->
-  <link name="upper_camera_link">
+  <!--<link name="upper_camera_link">
     <origin rpy="0 0 0" xyz="0 0 0"/>
   <inertial>
@@ -106,7 +106,7 @@
     <limit effort="10000" velocity="1000" lower="-1.57" upper="1.57"/>
     <joint_properties damping="1.0" friction="1.0" />
-  </joint>
+  </joint>-->
   <!-- camera -->
-  <gazebo reference="upper_camera_link">
+  <!--<gazebo reference="upper_camera_link">
     <sensor name="alphabot2_camera" type="camera" >
       <visualize>1</visualize>
@@ -130,7 +130,4 @@
         <noise>
           <type>gaussian</type>
-          <!-- Noise is sampled independently per pixel on each frame.
-               That pixel's noise value is added to each of its color
-               channels, which at that point lie in the range [0,1]. -->
           <mean>0.0</mean>
           <stddev>0.007</stddev>
@@ -152,4 +149,396 @@
       </plugin>
     </sensor>
+  </gazebo>-->
+  <joint name="sensor1_joint" type="fixed">
+    <axis xyz="0 1 0" />
+    <origin xyz="0.038 -0.028 -0.0242" rpy="0 0 0"/>
+    <parent link="link_chassis"/>
+    <child link="sensor1_bottom"/>
+  </joint>
+  <link name="sensor1_bottom">
+    <collision>
+      <origin xyz="0 0 0" rpy="0 0 0"/>
+      <geometry>
+    	<box size="0.005 0.006 0.0065"/>
+      </geometry>
+    </collision>
+    <visual>
+      <origin xyz="0 0 0" rpy="0 0 0"/>
+      <geometry>
+    	<box size="0.005 0.006 0.0065"/>
+      </geometry>
+    </visual>
+    <inertial>
+      <mass value="1e-5" />
+      <origin xyz="0 0 0" rpy="0 0 0"/>
+      <inertia ixx="1e-6" ixy="0" ixz="0" iyy="1e-6" iyz="0" izz="1e-6" />
+    </inertial>
+  </link>
+  <gazebo reference="sensor1_bottom">
+    <sensor type="ray" name="head_sensor1">
+      <pose>0 0 0 0 0 0</pose>
+      <visualize>true</visualize>
+      <update_rate>40</update_rate>
+      <ray>
+        <scan>
+          <vertical>
+            <samples>1</samples>
+            <resolution>1</resolution>
+            <min_angle>-1.5707963268</min_angle>
+            <max_angle>-1.5707963268</max_angle>
+          </vertical>
+        </scan>
+        <range>
+          <min>0.0010</min>
+          <max>0.20</max>
+          <resolution>0.01</resolution>
+        </range>
+        <noise>
+          <type>gaussian</type>
+          <mean>0.0</mean>
+          <stddev>0.01</stddev>
+        </noise>
+      </ray>
+      <plugin name="sensor1_controller" filename="libgazebo_ros_laser.so">
+        <topicName>/alphabot2/laser/scan/sensor1</topicName>
+        <frameName>sensor1_bottom</frameName>
+      </plugin>
+    </sensor>
+  </gazebo>
+  <joint name="sensor2_joint" type="fixed">
+    <axis xyz="0 1 0" />
+    <origin xyz="0.038  -0.014 -0.0242" rpy="0 0 0"/>
+    <parent link="link_chassis"/>
+    <child link="sensor2_bottom"/>
+  </joint>
+  <link name="sensor2_bottom">
+    <collision>
+      <origin xyz="0 0 0" rpy="0 0 0"/>
+      <geometry>
+    	<box size="0.005 0.006 0.0065"/>
+      </geometry>
+    </collision>
+    <visual>
+      <origin xyz="0 0 0" rpy="0 0 0"/>
+      <geometry>
+    	<box size="0.005 0.006 0.0065"/>
+      </geometry>
+    </visual>
+    <inertial>
+      <mass value="1e-5" />
+      <origin xyz="0 0 0" rpy="0 0 0"/>
+      <inertia ixx="1e-6" ixy="0" ixz="0" iyy="1e-6" iyz="0" izz="1e-6" />
+    </inertial>
+  </link>
+  <gazebo reference="sensor2_bottom">
+    <sensor type="ray" name="head_sensor2">
+      <pose>0 0 0 0 0 0</pose>
+      <visualize>true</visualize>
+      <update_rate>40</update_rate>
+      <ray>
+        <scan>
+          <vertical>
+            <samples>1</samples>
+            <resolution>1</resolution>
+            <min_angle>-1.5707963268</min_angle>
+            <max_angle>-1.5707963268</max_angle>
+          </vertical>
+        </scan>
+        <range>
+          <min>0.0010</min>
+          <max>0.20</max>
+          <resolution>0.01</resolution>
+        </range>
+        <noise>
+          <type>gaussian</type>
+          <mean>0.0</mean>
+          <stddev>0.01</stddev>
+        </noise>
+      </ray>
+      <plugin name="sensor2_controller" filename="libgazebo_ros_laser.so">
+        <topicName>/alphabot2/laser/scan/sensor2</topicName>
+        <frameName>sensor2_bottom</frameName>
+      </plugin>
+    </sensor>
+  </gazebo>
+  <joint name="sensor3_joint" type="fixed">
+    <axis xyz="0 1 0" />
+    <origin xyz="0.038 0 -0.0242" rpy="0 0 0"/>
+    <parent link="link_chassis"/>
+    <child link="sensor3_bottom"/>
+  </joint>
+  <link name="sensor3_bottom">
+    <collision>
+      <origin xyz="0 0 0" rpy="0 0 0"/>
+      <geometry>
+    	<box size="0.005 0.006 0.0065"/>
+      </geometry>
+    </collision>
+    <visual>
+      <origin xyz="0 0 0" rpy="0 0 0"/>
+      <geometry>
+    	<box size="0.005 0.006 0.0065"/>
+      </geometry>
+    </visual>
+    <inertial>
+      <mass value="1e-5" />
+      <origin xyz="0 0 0" rpy="0 0 0"/>
+      <inertia ixx="1e-6" ixy="0" ixz="0" iyy="1e-6" iyz="0" izz="1e-6" />
+    </inertial>
+  </link>
+  <gazebo reference="sensor3_bottom">
+    <sensor type="ray" name="head_sensor3">
+      <pose>0 0 0 0 0 0</pose>
+      <visualize>true</visualize>
+      <update_rate>40</update_rate>
+      <ray>
+        <scan>
+          <vertical>
+            <samples>1</samples>
+            <resolution>1</resolution>
+            <min_angle>-1.5707963268</min_angle>
+            <max_angle>-1.5707963268</max_angle>
+          </vertical>
+        </scan>
+        <range>
+          <min>0.0010</min>
+          <max>0.20</max>
+          <resolution>0.01</resolution>
+        </range>
+        <noise>
+          <type>gaussian</type>
+          <mean>0.0</mean>
+          <stddev>0.01</stddev>
+        </noise>
+      </ray>
+      <plugin name="sensor3_controller" filename="libgazebo_ros_laser.so">
+        <topicName>/alphabot2/laser/scan/sensor3</topicName>
+        <frameName>sensor3_bottom</frameName>
+      </plugin>
+    </sensor>
+  </gazebo>
+  <joint name="sensor4_joint" type="fixed">
+    <axis xyz="0 1 0" />
+    <origin xyz="0.038 0.014 -0.0242" rpy="0 0 0"/>
+    <parent link="link_chassis"/>
+    <child link="sensor4_bottom"/>
+  </joint>
+  <link name="sensor4_bottom">
+    <collision>
+      <origin xyz="0 0 0" rpy="0 0 0"/>
+      <geometry>
+    	<box size="0.005 0.006 0.0065"/>
+      </geometry>
+    </collision>
+    <visual>
+      <origin xyz="0 0 0" rpy="0 0 0"/>
+      <geometry>
+    	<box size="0.005 0.006 0.0065"/>
+      </geometry>
+    </visual>
+    <inertial>
+      <mass value="1e-5" />
+      <origin xyz="0 0 0" rpy="0 0 0"/>
+      <inertia ixx="1e-6" ixy="0" ixz="0" iyy="1e-6" iyz="0" izz="1e-6" />
+    </inertial>
+  </link>
+  <gazebo reference="sensor4_bottom">
+    <sensor type="ray" name="head_sensor4">
+      <pose>0 0 0 0 0 0</pose>
+      <visualize>true</visualize>
+      <update_rate>40</update_rate>
+      <ray>
+        <scan>
+          <vertical>
+            <samples>1</samples>
+            <resolution>1</resolution>
+            <min_angle>-1.5707963268</min_angle>
+            <max_angle>-1.5707963268</max_angle>
+          </vertical>
+        </scan>
+        <range>
+          <min>0.0010</min>
+          <max>0.20</max>
+          <resolution>0.01</resolution>
+        </range>
+        <noise>
+          <type>gaussian</type>
+          <mean>0.0</mean>
+          <stddev>0.01</stddev>
+        </noise>
+      </ray>
+      <plugin name="sensor4_controller" filename="libgazebo_ros_laser.so">
+        <topicName>/alphabot2/laser/scan/sensor4</topicName>
+        <frameName>sensor4_bottom</frameName>
+      </plugin>
+    </sensor>
+  </gazebo>
+  <joint name="sensor5_joint" type="fixed">
+    <axis xyz="0 1 0" />
+    <origin xyz="0.038 0.028 -0.0242" rpy="0 0 0"/>
+    <parent link="link_chassis"/>
+    <child link="sensor5_bottom"/>
+  </joint>
+  <link name="sensor5_bottom">
+    <collision>
+      <origin xyz="0 0 0" rpy="0 0 0"/>
+      <geometry>
+    	<box size="0.005 0.006 0.0065"/>
+      </geometry>
+    </collision>
+    <visual>
+      <origin xyz="0 0 0" rpy="0 0 0"/>
+      <geometry>
+    	<box size="0.005 0.006 0.0065"/>
+      </geometry>
+    </visual>
+    <inertial>
+      <mass value="1e-5" />
+      <origin xyz="0 0 0" rpy="0 0 0"/>
+      <inertia ixx="1e-6" ixy="0" ixz="0" iyy="1e-6" iyz="0" izz="1e-6" />
+    </inertial>
+  </link>
+  <gazebo reference="sensor5_bottom">
+    <sensor type="ray" name="head_sensor5">
+      <pose>0 0 0 0 0 0</pose>
+      <visualize>true</visualize>
+      <update_rate>40</update_rate>
+      <ray>
+        <scan>
+          <vertical>
+            <samples>1</samples>
+            <resolution>1</resolution>
+            <min_angle>-1.5707963268</min_angle>
+            <max_angle>-1.5707963268</max_angle>
+          </vertical>
+        </scan>
+        <range>
+          <min>0.0010</min>
+          <max>0.20</max>
+          <resolution>0.01</resolution>
+        </range>
+        <noise>
+          <type>gaussian</type>
+          <mean>0.0</mean>
+          <stddev>0.01</stddev>
+        </noise>
+      </ray>
+      <plugin name="sensor5_controller" filename="libgazebo_ros_laser.so">
+        <topicName>/alphabot2/laser/scan/sensor5</topicName>
+        <frameName>sensor5_bottom</frameName>
+      </plugin>
+    </sensor>
+  </gazebo>
+  <joint name="sensor1_top_joint" type="fixed">
+    <axis xyz="0 1 0" />
+    <origin xyz="0.0469 -0.022 0.0242" rpy="0 0 0"/>
+    <parent link="link_chassis"/>
+    <child link="sensor1_top"/>
+  </joint>
+  <link name="sensor1_top">
+    <collision>
+      <origin xyz="0 0 0" rpy="0 0 0"/>
+      <geometry>
+    	<box size="0.005 0.006 0.0065"/>
+      </geometry>
+    </collision>
+    <visual>
+      <origin xyz="0 0 0" rpy="0 0 0"/>
+      <geometry>
+    	<box size="0.005 0.006 0.0065"/>
+      </geometry>
+    </visual>
+    <inertial>
+      <mass value="1e-5" />
+      <origin xyz="0 0 0" rpy="0 0 0"/>
+      <inertia ixx="1e-6" ixy="0" ixz="0" iyy="1e-6" iyz="0" izz="1e-6" />
+    </inertial>
+  </link>
+  <gazebo reference="sensor1_top">
+    <sensor type="ray" name="head_sensor6">
+      <pose>0 0 0 0 0 0</pose>
+      <visualize>true</visualize>
+      <update_rate>40</update_rate>
+      <ray>
+        <scan>
+          <horizontal>
+            <samples>200</samples>
+            <resolution>1</resolution>
+            <min_angle>-1.5707963268</min_angle>
+            <max_angle>1.5707963268</max_angle>
+          </horizontal>
+        </scan>
+        <range>
+          <min>0.0010</min>
+          <max>3.0</max>
+          <resolution>0.01</resolution>
+        </range>
+        <noise>
+          <type>gaussian</type>
+          <mean>0.0</mean>
+          <stddev>0.01</stddev>
+        </noise>
+      </ray>
+      <plugin name="sensor1_top_controller" filename="libgazebo_ros_laser.so">
+        <topicName>/alphabot2/laser/scan/sensor1_top</topicName>
+        <frameName>sensor1_top</frameName>
+      </plugin>
+    </sensor>
+  </gazebo>
+  <joint name="sensor2_top_joint" type="fixed">
+    <axis xyz="0 1 0" />
+    <origin xyz="0.0469 0.022 0.0242" rpy="0 0 0"/>
+    <parent link="link_chassis"/>
+    <child link="sensor2_top"/>
+  </joint>
+  <link name="sensor2_top">
+    <collision>
+      <origin xyz="0 0 0" rpy="0 0 0"/>
+      <geometry>
+    	<box size="0.005 0.006 0.0065"/>
+      </geometry>
+    </collision>
+    <visual>
+      <origin xyz="0 0 0" rpy="0 0 0"/>
+      <geometry>
+    	<box size="0.005 0.006 0.0065"/>
+      </geometry>
+    </visual>
+    <inertial>
+      <mass value="1e-5" />
+      <origin xyz="0 0 0" rpy="0 0 0"/>
+      <inertia ixx="1e-6" ixy="0" ixz="0" iyy="1e-6" iyz="0" izz="1e-6" />
+    </inertial>
+  </link>
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
Commit message: Added Pan-Tilt control

File: alphabot2_world/robots/alphabot2.xacro (robot description, xacro)
@@ -50,16 +50,16 @@
   <!-- end of joint for left wheel -->
   <link name="lower_camera_link">
-  <inertial>
+    <inertial>
       <mass value="0.0225"/>
       <origin rpy="0 0 0" xyz="0 0 0"/>
       <inertia ixx="0.0000058388" ixy="0" ixz="0" iyy="0.0000063638" iyz="0" izz="0.0000046088"/>
-  </inertial>
-  <collision name="lower_camera_collision">
+    </inertial>
+    <collision name="lower_camera_collision">
       <origin rpy="0 0 0" xyz="0 0 0" />
       <geometry>
         <box size="0.037 0.033 0.045"/>
       </geometry>
-  </collision>
-  <visual name="lower_camera_visual">
+    </collision>
+    <visual name="lower_camera_visual">
       <origin rpy="0 0 0" xyz="0 0 0"/>
       <geometry>
@@ -67,7 +67,7 @@
       </geometry>
       <material name="red"/>
-  </visual>
+    </visual>
   </link>
-   <joint name="joint_lower_camera_link" type="continuous">
+  <joint name="joint_lower_camera" type="continuous"><!--AQUI USAM REVOLUTE https://answers.ros.org/question/142366/simulating-a-camera-with-a-pan-tilt-unit/-->
     <origin rpy="0 0 0" xyz="0 0 0.045"/>
     <child link="lower_camera_link" />
@@ -77,19 +77,31 @@
     <joint_properties damping="1.0" friction="1.0" />
   </joint>
+  <!--gazebo reference="lower_camera_link">
+        <material>Gazebo/Yellow</material>
+  </gazebo>
+  <transmission name="pan_trans">
+    <type>transmission_interface/SimpleTransmission</type>
+    <joint name="joint_lower_camera">
+      <hardwareInterface>EffortJointInterface</hardwareInterface>
+    </joint>
+    <actuator name="camera_pan_motor">
+      <mechanicalReduction>1</mechanicalReduction>
+    </actuator>
+  </transmission-->
   <!--TODO: plugin link da camara de baixo-->
   <link name="upper_camera_link">
     <origin rpy="0 0 0" xyz="0 0 0"/>
-  <inertial>
+    <inertial>
       <mass value="0.0225"/>
       <origin rpy="0 ${3.14/2} 0" xyz="0 0 0 "/>
       <inertia ixx="0" ixy="0" ixz="0" iyy="0.000006" iyz="0" izz="0.000005"/>
-  </inertial>
-  <collision name="upper_camera_collision">
+    </inertial>
+    <collision name="upper_camera_collision">
       <origin rpy="0 ${3.14/2} 0" xyz="0 0 0" />
       <geometry>
         <mesh filename="package://alphabot2_world/meshes/chassis.stl" />
       </geometry>
-  </collision>
-  <visual name="upper_camera_visual">
+    </collision>
+    <visual name="upper_camera_visual">
       <origin rpy="0 ${3.14/2} 0" xyz="0 0 0"/>
       <geometry>
@@ -97,8 +109,8 @@
       </geometry>
       <material name="blue"/>
-  </visual>
+    </visual>
   </link>
-   <joint name="joint_upper_camera_link" type="continuous">
-    <origin rpy="0 ${-3.14/2} 0" xyz="0 0 0.045"/>
+  <joint name="joint_upper_camera" type="continuous">
+    <origin rpy="0 ${-3.14/2} 0" xyz="0 0 0.045"/> <!--0.045-->
     <child link="upper_camera_link" />
     <parent link="lower_camera_link"/>
@@ -107,6 +119,33 @@
     <joint_properties damping="1.0" friction="1.0" />
   </joint>
+  <!--gazebo reference="upper_camera_link">
+        <material>Gazebo/Yellow</material>
+  </gazebo>
+  <transmission name="tilt_trans">
+    <type>transmission_interface/SimpleTransmission</type>
+    <joint name="joint_upper_camera">
+      <hardwareInterface>EffortJointInterface</hardwareInterface>
+    </joint>
+    <actuator name="camera_tilt_motor">
+      <mechanicalReduction>1</mechanicalReduction>
+    </actuator>
+  </transmission-->
+  <!--For all the transmission tags-->
+  <!--gazebo>
+    <plugin name="gazebo_ros_control" filename="libgazebo_ros_control.so">
+      <robotNamespace>/alphabot2</robotNamespace>
+    </plugin>
+  </gazebo-->
   <!-- camera -->
-  <gazebo reference="upper_camera_link">
+  <joint name="joint_camera" type="fixed">
+    <origin rpy="0 0 0" xyz="0 0 0.08"/>
+    <child link="camera_link" />
+    <parent link="upper_camera_link"/>
+    <limit effort="10000" velocity="1000"/>
+    <joint_properties damping="1.0" friction="1.0" />
+  </joint>
+  <link name="camera_link">
+  </link>
+  <gazebo reference="camera_link">
     <sensor name="alphabot2_camera" type="camera" >
       <visualize>1</visualize>
@@ -125,5 +164,5 @@
         </image>
         <clip>
-          <near>0.01</near>
+          <near>7</near>
           <far>1000</far>
         </clip>

File: alphabot2_world/robots/gazebo.xacro (robot description, xacro)
@@ -10,4 +10,7 @@
   <gazebo reference="link_right_wheel">
     <material>Gazebo/Black</material>
+  </gazebo>
+  <gazebo reference="upper_camera_link">
+    <material>Gazebo/Blue</material>
   </gazebo>
   <!-- end of gazebo colors definitions -->

Commit message: Add trasmission message

File: alphabot2_world/robots/alphabot2.xacro (robot description, xacro)
@@ -69,5 +69,5 @@
     </visual>
   </link>
-  <joint name="joint_lower_camera" type="continuous"><!--AQUI USAM REVOLUTE https://answers.ros.org/question/142366/simulating-a-camera-with-a-pan-tilt-unit/-->
+  <joint name="joint_lower_camera_link" type="continuous"><!--AQUI USAM REVOLUTE https://answers.ros.org/question/142366/simulating-a-camera-with-a-pan-tilt-unit/-->
     <origin rpy="0 0 0" xyz="0 0 0.045"/>
     <child link="lower_camera_link" />
@@ -77,5 +77,5 @@
     <joint_properties damping="1.0" friction="1.0" />
   </joint>
-  <!--gazebo reference="lower_camera_link">
+  <gazebo reference="lower_camera_link">
         <material>Gazebo/Yellow</material>
   </gazebo>
@@ -88,5 +88,5 @@
       <mechanicalReduction>1</mechanicalReduction>
     </actuator>
-  </transmission-->
+  </transmission>
   <!--TODO: plugin link da camara de baixo-->
   <link name="upper_camera_link">
@@ -111,5 +111,5 @@
     </visual>
   </link>
-  <joint name="joint_upper_camera" type="continuous">
+  <joint name="joint_upper_camera_link" type="continuous">
     <origin rpy="0 ${-3.14/2} 0" xyz="0 0 0.045"/> <!--0.045-->
     <child link="upper_camera_link" />
@@ -119,10 +119,10 @@
     <joint_properties damping="1.0" friction="1.0" />
   </joint>
-  <!--gazebo reference="upper_camera_link">
+  <gazebo reference="upper_camera_link">
         <material>Gazebo/Yellow</material>
   </gazebo>
   <transmission name="tilt_trans">
     <type>transmission_interface/SimpleTransmission</type>
-    <joint name="joint_upper_camera">
+    <joint name="joint_upper_camera_link">
       <hardwareInterface>EffortJointInterface</hardwareInterface>
     </joint>
@@ -130,22 +130,13 @@
       <mechanicalReduction>1</mechanicalReduction>
     </actuator>
-  </transmission-->
+  </transmission>
   <!--For all the transmission tags-->
-  <!--gazebo>
+  <gazebo>
     <plugin name="gazebo_ros_control" filename="libgazebo_ros_control.so">
       <robotNamespace>/alphabot2</robotNamespace>
     </plugin>
-  </gazebo-->
+  </gazebo>
   <!-- camera -->
-  <joint name="joint_camera" type="fixed">
-    <origin rpy="0 0 0" xyz="0 0 0.08"/>
-    <child link="camera_link" />
-    <parent link="upper_camera_link"/>
-    <limit effort="10000" velocity="1000"/>
-    <joint_properties damping="1.0" friction="1.0" />
-  </joint>
-  <link name="camera_link">
-  </link>
-  <gazebo reference="camera_link">
+  <gazebo reference="upper_camera_link">
     <sensor name="alphabot2_camera" type="camera" >
       <visualize>1</visualize>
@@ -164,5 +155,5 @@
         </image>
         <clip>
-          <near>7</near>
+          <near>0.01</near>
           <far>1000</far>
         </clip>

Commit message: Fixing tramissions link names

File: alphabot2_world/robots/alphabot2.xacro (robot description, xacro)
@@ -82,5 +82,5 @@
   <transmission name="pan_trans">
     <type>transmission_interface/SimpleTransmission</type>
-    <joint name="joint_lower_camera">
+    <joint name="joint_lower_camera_link">
       <hardwareInterface>EffortJointInterface</hardwareInterface>
     </joint>
