Commit message: Change Alphabot links from stl to geometry

File: alphabot2_world/robots/alphabot2.xacro (robot description, xacro)
@@ -22,7 +22,7 @@
     </collision>
     <visual>
-      <origin rpy="0 0 0" xyz="0 0 -0.0225"/>
+      <origin rpy="0 0 0" xyz="0 0 -0.0065"/>
       <geometry>
-        <mesh filename="package://alphabot2_world/meshes/chassis.stl" />
+        <cylinder radius="0.055" length="0.045"/>
       </geometry>
       <material name="blue"/>
@@ -49,4 +49,5 @@
   <xacro:joint_wheel name="joint_left_wheel"   child="link_left_wheel"   origin_xyz="0 -0.046 -0.016"  />
   <!-- end of joint for left wheel -->
+  <!-- Lower Camera-->
   <link name="lower_camera_link">
     <inertial>
@@ -56,5 +57,5 @@
     </inertial>
     <collision name="lower_camera_collision">
-      <origin rpy="0 0 0" xyz="0 0 0" />
+      <origin rpy="0 0 0" xyz="0 0 0.0225" />
       <geometry>
         <box size="0.037 0.033 0.045"/>
@@ -69,11 +70,11 @@
     </visual>
   </link>
-  <joint name="joint_lower_camera_link" type="continuous"><!--AQUI USAM REVOLUTE https://answers.ros.org/question/142366/simulating-a-camera-with-a-pan-tilt-unit/-->
-    <origin rpy="0 0 0" xyz="0 0 0.045"/>
+  <joint name="joint_lower_camera_link" type="revolute"><!--AQUI USAM REVOLUTE -->
+    <origin rpy="0 0 0" xyz="0 0 0.0225"/>
     <child link="lower_camera_link" />
     <parent link="link_chassis"/>
     <axis rpy="0 0 0" xyz="0 0 1"/>
-    <limit effort="10000" velocity="1000" lower="-1.57" upper="1.57"/>
-    <joint_properties damping="1.0" friction="1.0" />
+    <limit effort="90" velocity="1.396" lower="-1.57" upper="1.57"/>
+    <dynamics dampling="2" friction="1"/>
   </joint>
   <gazebo reference="lower_camera_link">
@@ -82,6 +83,6 @@
   <transmission name="pan_trans">
     <type>transmission_interface/SimpleTransmission</type>
-    <joint name="joint_lower_camera">
-      <hardwareInterface>EffortJointInterface</hardwareInterface>
+    <joint name="joint_lower_camera_link">
+      <hardwareInterface>hardware_interface/EffortJointInterface</hardwareInterface>
     </joint>
     <actuator name="camera_pan_motor">
@@ -89,5 +90,6 @@
     </actuator>
   </transmission>
-  <!--TODO: plugin link da camara de baixo-->
+  <!--End Lower Camera-->
+  <!--Upper Camera-->
   <link name="upper_camera_link">
     <origin rpy="0 0 0" xyz="0 0 0"/>
@@ -100,5 +102,5 @@
       <origin rpy="0 ${3.14/2} 0" xyz="0 0 0" />
       <geometry>
-        <mesh filename="package://alphabot2_world/meshes/chassis.stl" />
+        <box size="0.037 0.033 0.045"/>
       </geometry>
     </collision>
@@ -106,24 +108,24 @@
       <origin rpy="0 ${3.14/2} 0" xyz="0 0 0"/>
       <geometry>
-        <mesh filename="package://alphabot2_world/meshes/camera.stl" />
+        <box size="0.037 0.033 0.045"/>
       </geometry>
       <material name="blue"/>
     </visual>
   </link>
-  <joint name="joint_upper_camera_link" type="continuous">
+  <gazebo reference="upper_camera_link">
+        <material>Gazebo/Yellow</material>
+  </gazebo>
+  <joint name="joint_upper_camera_link" type="revolute">
     <origin rpy="0 ${-3.14/2} 0" xyz="0 0 0.045"/> <!--0.045-->
     <child link="upper_camera_link" />
     <parent link="lower_camera_link"/>
     <axis rpy="0 0 0" xyz="0 1 0"/>
-    <limit effort="10000" velocity="1000" lower="-1.57" upper="1.57"/>
-    <joint_properties damping="1.0" friction="1.0" />
+    <limit effort="90" velocity="1.396" lower="-1.57" upper="1.57"/>
+    <dynamics dampling="2" friction="1"/>
   </joint>
-  <gazebo reference="upper_camera_link">
-        <material>Gazebo/Yellow</material>
-  </gazebo>
   <transmission name="tilt_trans">
     <type>transmission_interface/SimpleTransmission</type>
     <joint name="joint_upper_camera_link">
-      <hardwareInterface>EffortJointInterface</hardwareInterface>
+      <hardwareInterface>hardware_interface/EffortJointInterface</hardwareInterface>
     </joint>
     <actuator name="camera_tilt_motor">
@@ -131,4 +133,5 @@
     </actuator>
   </transmission>
+  <!--End Upper Camera-->
   <!--For all the transmission tags-->
   <gazebo>

Commit message: Stl to Geometry

File: alphabot2_world/robots/alphabot2.xacro (robot description, xacro)
@@ -57,5 +57,5 @@
     </inertial>
     <collision name="lower_camera_collision">
-      <origin rpy="0 0 0" xyz="0 0 0.0225" />
+      <origin rpy="0 0 0" xyz="0 0 0" />
       <geometry>
         <box size="0.037 0.033 0.045"/>
@@ -71,5 +71,5 @@
   </link>
   <joint name="joint_lower_camera_link" type="revolute"><!--AQUI USAM REVOLUTE -->
-    <origin rpy="0 0 0" xyz="0 0 0.0225"/>
+    <origin rpy="0 0 0" xyz="0 0 0.045"/>
     <child link="lower_camera_link" />
     <parent link="link_chassis"/>

Commit message: Detect lines in camera image

File: alphabot2_world/robots/alphabot2.xacro (robot description, xacro)
@@ -76,8 +76,10 @@
     <axis rpy="0 0 0" xyz="0 0 1"/>
     <limit effort="90" velocity="1.396" lower="-1.57" upper="1.57"/>
-    <dynamics dampling="2" friction="1"/>
+    <dynamics dampling="0" friction="0"/>
   </joint>
   <gazebo reference="lower_camera_link">
         <material>Gazebo/Yellow</material>
+        <selfCollide>true</selfCollide>
+        <turnGravityOff>true</turnGravityOff>
   </gazebo>
   <transmission name="pan_trans">
@@ -115,4 +117,6 @@
   <gazebo reference="upper_camera_link">
         <material>Gazebo/Yellow</material>
+        <selfCollide>true</selfCollide>
+        <turnGravityOff>true</turnGravityOff>
   </gazebo>
   <joint name="joint_upper_camera_link" type="revolute">
@@ -122,5 +126,5 @@
     <axis rpy="0 0 0" xyz="0 1 0"/>
     <limit effort="90" velocity="1.396" lower="-1.57" upper="1.57"/>
-    <dynamics dampling="2" friction="1"/>
+    <dynamics dampling="0" friction="0"/>
   </joint>
   <transmission name="tilt_trans">

Commit message: Fix pan joint

File: alphabot2_world/robots/alphabot2.xacro (robot description, xacro)
@@ -70,21 +70,21 @@
     </visual>
   </link>
-  <joint name="joint_lower_camera_link" type="revolute"><!--AQUI USAM REVOLUTE -->
+  <joint name="joint_lower_camera_link" type="continuous"><!--AQUI USAM REVOLUTE -->
     <origin rpy="0 0 0" xyz="0 0 0.045"/>
     <child link="lower_camera_link" />
     <parent link="link_chassis"/>
     <axis rpy="0 0 0" xyz="0 0 1"/>
-    <limit effort="90" velocity="1.396" lower="-1.57" upper="1.57"/>
-    <dynamics dampling="0" friction="0"/>
+    <limit effort="30" velocity="1" lower="-1.57" upper="1.57"/>
+    <dynamics dampling="2" friction="2"/>
   </joint>
   <gazebo reference="lower_camera_link">
         <material>Gazebo/Yellow</material>
-        <selfCollide>true</selfCollide>
-        <turnGravityOff>true</turnGravityOff>
+        <!--selfCollide>false</selfCollide>
+        <turnGravityOff>true</turnGravityOff-->
   </gazebo>
   <transmission name="pan_trans">
     <type>transmission_interface/SimpleTransmission</type>
     <joint name="joint_lower_camera_link">
-      <hardwareInterface>hardware_interface/EffortJointInterface</hardwareInterface>
+      <hardwareInterface>PositionJointInterface</hardwareInterface>
     </joint>
     <actuator name="camera_pan_motor">
@@ -117,6 +117,6 @@
   <gazebo reference="upper_camera_link">
         <material>Gazebo/Yellow</material>
-        <selfCollide>true</selfCollide>
-        <turnGravityOff>true</turnGravityOff>
+        <!--selfCollide>true</selfCollide>
+        <turnGravityOff>true</turnGravityOff-->
   </gazebo>
   <joint name="joint_upper_camera_link" type="revolute">
@@ -125,6 +125,6 @@
     <parent link="lower_camera_link"/>
     <axis rpy="0 0 0" xyz="0 1 0"/>
-    <limit effort="90" velocity="1.396" lower="-1.57" upper="1.57"/>
-    <dynamics dampling="0" friction="0"/>
+    <limit effort="30" velocity="1" lower="-1.57" upper="1.57"/>
+    <dynamics dampling="2" friction="2"/>
   </joint>
   <transmission name="tilt_trans">
@@ -138,5 +138,5 @@
   </transmission>
   <!--End Upper Camera-->
-  <!--For all the transmission tags-->
+  <!--For all the transmission tags; links gazebo with ROS-->
   <gazebo>
     <plugin name="gazebo_ros_control" filename="libgazebo_ros_control.so">

Commit message: modified sensors (for the last time!)

File: alphabot2_world/robots/alphabot2.xacro (robot description, xacro)
@@ -152,5 +152,5 @@
   <joint name="sensor1_joint" type="fixed">
     <axis xyz="0 1 0" />
-    <origin xyz="0.038 -0.028 -0.0242" rpy="0 0 0"/>
+    <origin xyz="0.038 -0.028 -0.0242" rpy="0 1.57 0"/>
     <parent link="link_chassis"/>
     <child link="sensor1_bottom"/>
@@ -176,31 +176,42 @@
   </link>
   <gazebo reference="sensor1_bottom">
-    <sensor type="ray" name="head_sensor1">
-      <pose>0 0 0 0 0 0</pose>
-      <visualize>true</visualize>
-      <update_rate>40</update_rate>
-      <ray>
-        <scan>
-          <vertical>
-            <samples>1</samples>
-            <resolution>1</resolution>
-            <min_angle>-1.5707963268</min_angle>
-            <max_angle>-1.5707963268</max_angle>
-          </vertical>
-        </scan>
-        <range>
-          <min>0.0010</min>
-          <max>0.20</max>
-          <resolution>0.01</resolution>
-        </range>
-        <noise>
-          <type>gaussian</type>
-          <mean>0.0</mean>
-          <stddev>0.01</stddev>
-        </noise>
-      </ray>
-      <plugin name="sensor1_controller" filename="libgazebo_ros_laser.so">
-        <topicName>/alphabot2/laser/scan/sensor1</topicName>
+    <sensor name="sensor1_bottom" type="camera" >
+      <visualize>1</visualize>
+      <always_on>1</always_on>
+      <update_rate>40.0</update_rate>
+      <camera name="sensor1_bottom">
+      <origin rpy="0 0 0" xyz="0 0 0"/>
+        <horizontal_fov>1.08504</horizontal_fov>
+        <image>
+          <width>100</width>
+          <height>100</height>
+          <format>R8G8B8</format>
+        </image>
+        <clip>
+          <near>0.001</near>
+          <far>5</far>
+        </clip>
+        <noise>
+          <type>gaussian</type>
+          <!-- Noise is sampled independently per pixel on each frame.
+               That pixel's noise value is added to each of its color
+               channels, which at that point lie in the range [0,1]. -->
+          <mean>0.0</mean>
+          <stddev>0.007</stddev>
+        </noise>
+      </camera>
+      <plugin name="camera_controller" filename="libgazebo_ros_camera.so">
+        <alwaysOn>true</alwaysOn>
+        <updateRate>40.0</updateRate>
+        <cameraName>sensor1_cam/</cameraName>
+        <imageTopicName>image_raw</imageTopicName>
+        <cameraInfoTopicName>camera_info</cameraInfoTopicName>
         <frameName>sensor1_bottom</frameName>
+        <hackBaseline>0.07</hackBaseline>
+        <distortionK1>0.0</distortionK1>
+        <distortionK2>0.0</distortionK2>
+        <distortionK3>0.0</distortionK3>
+        <distortionT1>0.0</distortionT1>
+        <distortionT2>0.0</distortionT2>
       </plugin>
     </sensor>
@@ -208,5 +219,5 @@
   <joint name="sensor2_joint" type="fixed">
     <axis xyz="0 1 0" />
-    <origin xyz="0.038  -0.014 -0.0242" rpy="0 0 0"/>
+    <origin xyz="0.038  -0.014 -0.0242" rpy="0 1.57 0"/>
     <parent link="link_chassis"/>
     <child link="sensor2_bottom"/>
@@ -232,31 +243,42 @@
   </link>
   <gazebo reference="sensor2_bottom">
-    <sensor type="ray" name="head_sensor2">
-      <pose>0 0 0 0 0 0</pose>
-      <visualize>true</visualize>
-      <update_rate>40</update_rate>
-      <ray>
-        <scan>
-          <vertical>
-            <samples>1</samples>
-            <resolution>1</resolution>
-            <min_angle>-1.5707963268</min_angle>
-            <max_angle>-1.5707963268</max_angle>
-          </vertical>
-        </scan>
-        <range>
-          <min>0.0010</min>
-          <max>0.20</max>
-          <resolution>0.01</resolution>
-        </range>
-        <noise>
-          <type>gaussian</type>
-          <mean>0.0</mean>
-          <stddev>0.01</stddev>
-        </noise>
-      </ray>
-      <plugin name="sensor2_controller" filename="libgazebo_ros_laser.so">
-        <topicName>/alphabot2/laser/scan/sensor2</topicName>
+    <sensor name="sensor2_bottom" type="camera" >
+      <visualize>1</visualize>
+      <always_on>1</always_on>
+      <update_rate>40.0</update_rate>
+      <camera name="sensor2_bottom">
+      <origin rpy="0 0 0" xyz="0 0 0"/>
+        <horizontal_fov>1.08504</horizontal_fov>
+        <image>
+          <width>100</width>
+          <height>100</height>
+          <format>R8G8B8</format>
+        </image>
+        <clip>
+          <near>0.001</near>
+          <far>5</far>
+        </clip>
+        <noise>
+          <type>gaussian</type>
+          <!-- Noise is sampled independently per pixel on each frame.
+               That pixel's noise value is added to each of its color
+               channels, which at that point lie in the range [0,1]. -->
+          <mean>0.0</mean>
+          <stddev>0.007</stddev>
+        </noise>
+      </camera>
+      <plugin name="camera_controller" filename="libgazebo_ros_camera.so">
+        <alwaysOn>true</alwaysOn>
+        <updateRate>40.0</updateRate>
+        <cameraName>sensor2_bottom/</cameraName>
+        <imageTopicName>image_raw</imageTopicName>
+        <cameraInfoTopicName>camera_info</cameraInfoTopicName>
         <frameName>sensor2_bottom</frameName>
+        <hackBaseline>0.07</hackBaseline>
+        <distortionK1>0.0</distortionK1>
+        <distortionK2>0.0</distortionK2>
+        <distortionK3>0.0</distortionK3>
+        <distortionT1>0.0</distortionT1>
+        <distortionT2>0.0</distortionT2>
       </plugin>
     </sensor>
@@ -264,5 +286,5 @@
   <joint name="sensor3_joint" type="fixed">
     <axis xyz="0 1 0" />
-    <origin xyz="0.038 0 -0.0242" rpy="0 0 0"/>
+    <origin xyz="0.038 0 -0.0242" rpy="0 1.57 0"/>
     <parent link="link_chassis"/>
     <child link="sensor3_bottom"/>
@@ -288,31 +310,42 @@
   </link>
   <gazebo reference="sensor3_bottom">
-    <sensor type="ray" name="head_sensor3">
-      <pose>0 0 0 0 0 0</pose>
-      <visualize>true</visualize>
-      <update_rate>40</update_rate>
-      <ray>
-        <scan>
-          <vertical>
-            <samples>1</samples>
-            <resolution>1</resolution>
-            <min_angle>-1.5707963268</min_angle>
-            <max_angle>-1.5707963268</max_angle>
-          </vertical>
-        </scan>
-        <range>
-          <min>0.0010</min>
-          <max>0.20</max>
-          <resolution>0.01</resolution>
-        </range>
-        <noise>
-          <type>gaussian</type>
-          <mean>0.0</mean>
-          <stddev>0.01</stddev>
-        </noise>
-      </ray>
-      <plugin name="sensor3_controller" filename="libgazebo_ros_laser.so">
-        <topicName>/alphabot2/laser/scan/sensor3</topicName>
+    <sensor name="sensor3_bottom" type="camera" >
+      <visualize>1</visualize>
+      <always_on>1</always_on>
+      <update_rate>40.0</update_rate>
+      <camera name="sensor3_bottom">
+      <origin rpy="0 0 0" xyz="0 0 0"/>
+        <horizontal_fov>1.08504</horizontal_fov>
+        <image>
+          <width>100</width>
+          <height>100</height>
+          <format>R8G8B8</format>
+        </image>
+        <clip>
+          <near>0.001</near>
+          <far>5</far>
+        </clip>
+        <noise>
+          <type>gaussian</type>
+          <!-- Noise is sampled independently per pixel on each frame.
+               That pixel's noise value is added to each of its color
+               channels, which at that point lie in the range [0,1]. -->
+          <mean>0.0</mean>
+          <stddev>0.007</stddev>
+        </noise>
+      </camera>
+      <plugin name="camera_controller" filename="libgazebo_ros_camera.so">
+        <alwaysOn>true</alwaysOn>
+        <updateRate>40.0</updateRate>
+        <cameraName>sensor3_bottom/</cameraName>
+        <imageTopicName>image_raw</imageTopicName>
+        <cameraInfoTopicName>camera_info</cameraInfoTopicName>
         <frameName>sensor3_bottom</frameName>
+        <hackBaseline>0.07</hackBaseline>
+        <distortionK1>0.0</distortionK1>
+        <distortionK2>0.0</distortionK2>
+        <distortionK3>0.0</distortionK3>
+        <distortionT1>0.0</distortionT1>
+        <distortionT2>0.0</distortionT2>
       </plugin>
     </sensor>
@@ -320,5 +353,5 @@
   <joint name="sensor4_joint" type="fixed">
     <axis xyz="0 1 0" />
-    <origin xyz="0.038 0.014 -0.0242" rpy="0 0 0"/>
+    <origin xyz="0.038 0.014 -0.0242" rpy="0 1.57 0"/>
     <parent link="link_chassis"/>
     <child link="sensor4_bottom"/>
@@ -344,31 +377,42 @@
   </link>
   <gazebo reference="sensor4_bottom">
-    <sensor type="ray" name="head_sensor4">
-      <pose>0 0 0 0 0 0</pose>
-      <visualize>true</visualize>
-      <update_rate>40</update_rate>
-      <ray>
-        <scan>
-          <vertical>
-            <samples>1</samples>
-            <resolution>1</resolution>
-            <min_angle>-1.5707963268</min_angle>
-            <max_angle>-1.5707963268</max_angle>
-          </vertical>
-        </scan>
-        <range>
-          <min>0.0010</min>
-          <max>0.20</max>
-          <resolution>0.01</resolution>
-        </range>
-        <noise>
-          <type>gaussian</type>
-          <mean>0.0</mean>
-          <stddev>0.01</stddev>
-        </noise>
-      </ray>
-      <plugin name="sensor4_controller" filename="libgazebo_ros_laser.so">
-        <topicName>/alphabot2/laser/scan/sensor4</topicName>
+    <sensor name="sensor4_bottom" type="camera" >
+      <visualize>1</visualize>
+      <always_on>1</always_on>
+      <update_rate>40.0</update_rate>
+      <camera name="sensor4_bottom">
+      <origin rpy="0 0 0" xyz="0 0 0"/>
+        <horizontal_fov>1.08504</horizontal_fov>
+        <image>
+          <width>100</width>
+          <height>100</height>
+          <format>R8G8B8</format>
+        </image>
+        <clip>
+          <near>0.001</near>
+          <far>5</far>
+        </clip>
+        <noise>
+          <type>gaussian</type>
+          <!-- Noise is sampled independently per pixel on each frame.
+               That pixel's noise value is added to each of its color
+               channels, which at that point lie in the range [0,1]. -->
+          <mean>0.0</mean>
+          <stddev>0.007</stddev>
+        </noise>
+      </camera>
+      <plugin name="camera_controller" filename="libgazebo_ros_camera.so">
+        <alwaysOn>true</alwaysOn>
+        <updateRate>40.0</updateRate>
+        <cameraName>sensor4_bottom/</cameraName>
+        <imageTopicName>image_raw</imageTopicName>
+        <cameraInfoTopicName>camera_info</cameraInfoTopicName>
         <frameName>sensor4_bottom</frameName>
+        <hackBaseline>0.07</hackBaseline>
+        <distortionK1>0.0</distortionK1>
+        <distortionK2>0.0</distortionK2>
+        <distortionK3>0.0</distortionK3>
+        <distortionT1>0.0</distortionT1>
+        <distortionT2>0.0</distortionT2>
       </plugin>
     </sensor>
@@ -376,5 +420,5 @@
   <joint name="sensor5_joint" type="fixed">
     <axis xyz="0 1 0" />
-    <origin xyz="0.038 0.028 -0.0242" rpy="0 0 0"/>
+    <origin xyz="0.038 0.028 -0.0242" rpy="0 1.57 0"/>
     <parent link="link_chassis"/>
     <child link="sensor5_bottom"/>
@@ -400,31 +444,42 @@
   </link>
   <gazebo reference="sensor5_bottom">
-    <sensor type="ray" name="head_sensor5">
-      <pose>0 0 0 0 0 0</pose>
-      <visualize>true</visualize>
-      <update_rate>40</update_rate>
-      <ray>
-        <scan>
-          <vertical>
-            <samples>1</samples>
-            <resolution>1</resolution>
-            <min_angle>-1.5707963268</min_angle>
-            <max_angle>-1.5707963268</max_angle>
-          </vertical>
-        </scan>
-        <range>
-          <min>0.0010</min>
-          <max>0.20</max>
-          <resolution>0.01</resolution>
-        </range>
-        <noise>
-          <type>gaussian</type>
-          <mean>0.0</mean>
-          <stddev>0.01</stddev>
-        </noise>
-      </ray>
-      <plugin name="sensor5_controller" filename="libgazebo_ros_laser.so">
-        <topicName>/alphabot2/laser/scan/sensor5</topicName>
+    <sensor name="sensor5_bottom" type="camera" >
+      <visualize>1</visualize>
+      <always_on>1</always_on>
+      <update_rate>40.0</update_rate>
+      <camera name="sensor5_bottom">
+      <origin rpy="0 0 0" xyz="0 0 0"/>
+        <horizontal_fov>1.08504</horizontal_fov>
+        <image>
+          <width>100</width>
+          <height>100</height>
+          <format>R8G8B8</format>
+        </image>
+        <clip>
+          <near>0.001</near>
+          <far>5</far>
+        </clip>
+        <noise>
+          <type>gaussian</type>
+          <!-- Noise is sampled independently per pixel on each frame.
+               That pixel's noise value is added to each of its color
+               channels, which at that point lie in the range [0,1]. -->
+          <mean>0.0</mean>
+          <stddev>0.007</stddev>
+        </noise>
+      </camera>
+      <plugin name="camera_controller" filename="libgazebo_ros_camera.so">
+        <alwaysOn>true</alwaysOn>
+        <updateRate>40.0</updateRate>
+        <cameraName>sensor5_bottom/</cameraName>
+        <imageTopicName>image_raw</imageTopicName>
+        <cameraInfoTopicName>camera_info</cameraInfoTopicName>
         <frameName>sensor5_bottom</frameName>
+        <hackBaseline>0.07</hackBaseline>
+        <distortionK1>0.0</distortionK1>
+        <distortionK2>0.0</distortionK2>
+        <distortionK3>0.0</distortionK3>
+        <distortionT1>0.0</distortionT1>
+        <distortionT2>0.0</distortionT2>
       </plugin>
     </sensor>
@@ -432,5 +487,5 @@
   <joint name="sensor1_top_joint" type="fixed">
     <axis xyz="0 1 0" />
-    <origin xyz="0.0469 -0.022 0.0242" rpy="0 0 0"/>
+    <origin xyz="0.0469 -0.022 -0.0183" rpy="0 0 0"/>
     <parent link="link_chassis"/>
     <child link="sensor1_top"/>
@@ -488,5 +543,5 @@
   <joint name="sensor2_top_joint" type="fixed">
     <axis xyz="0 1 0" />
-    <origin xyz="0.0469 0.022 0.0242" rpy="0 0 0"/>
+    <origin xyz="0.0469 0.022 -0.0183" rpy="0 0 0"/>
     <parent link="link_chassis"/>
     <child link="sensor2_top"/>
