Commit message: Pan.tilt fix

File: alphabot2_world/robots/alphabot2.xacro (robot description, xacro)
@@ -98,9 +98,9 @@
     <inertial>
       <mass value="0.0225"/>
-      <origin rpy="0 ${3.14/2} 0" xyz="0 0 0 "/>
-      <inertia ixx="0" ixy="0" ixz="0" iyy="0.000006" iyz="0" izz="0.000005"/>
+      <origin rpy="0 0 0" xyz="0 0 0 "/>
+      <inertia ixx="0.0000058388" ixy="0" ixz="0" iyy="0.0000063638" iyz="0" izz="0.0000046088"/>
     </inertial>
     <collision name="upper_camera_collision">
-      <origin rpy="0 ${3.14/2} 0" xyz="0 0 0" />
+      <origin rpy="0 0 0" xyz="0 0 0" />
       <geometry>
         <box size="0.037 0.033 0.045"/>
@@ -108,5 +108,5 @@
     </collision>
     <visual name="upper_camera_visual">
-      <origin rpy="0 ${3.14/2} 0" xyz="0 0 0"/>
+      <origin rpy="0 0 0" xyz="0 0 0"/>
       <geometry>
         <box size="0.037 0.033 0.045"/>
@@ -121,5 +121,5 @@
   </gazebo>
   <joint name="joint_upper_camera_link" type="revolute">
-    <origin rpy="0 ${-3.14/2} 0" xyz="0 0 0.045"/> <!--0.045-->
+    <origin rpy="0 0 0" xyz="0 0 0.045"/> <!--0.045-->
     <child link="upper_camera_link" />
     <parent link="lower_camera_link"/>
@@ -131,5 +131,5 @@
     <type>transmission_interface/SimpleTransmission</type>
     <joint name="joint_upper_camera_link">
-      <hardwareInterface>hardware_interface/EffortJointInterface</hardwareInterface>
+      <hardwareInterface>PositionJointInterface</hardwareInterface>
     </joint>
     <actuator name="camera_tilt_motor">

Commit message: started code for top sensors

File: alphabot2_world/robots/alphabot2.xacro (robot description, xacro)
@@ -18,5 +18,5 @@
     <collision name="collision_chassis">
       <geometry>
-        <cylinder radius="0.055" length="0.045"/>
+        <mesh filename="package://alphabot2_world/meshes/chassis.stl" />
       </geometry>
     </collision>
@@ -492,10 +492,4 @@
   </joint>
   <link name="sensor1_top">
-    <collision>
-      <origin xyz="0 0 0" rpy="0 0 0"/>
-      <geometry>
-    	<box size="0.005 0.006 0.0065"/>
-      </geometry>
-    </collision>
     <visual>
       <origin xyz="0 0 0" rpy="0 0 0"/>
@@ -518,13 +512,13 @@
         <scan>
           <horizontal>
-            <samples>200</samples>
+            <samples>100</samples>
             <resolution>1</resolution>
-            <min_angle>-1.5707963268</min_angle>
-            <max_angle>1.5707963268</max_angle>
+            <min_angle>-0.785398163</min_angle>
+            <max_angle>0.785398163</max_angle>
           </horizontal>
         </scan>
         <range>
           <min>0.0010</min>
-          <max>3.0</max>
+          <max>0.3</max>
           <resolution>0.01</resolution>
         </range>
@@ -548,10 +542,4 @@
   </joint>
   <link name="sensor2_top">
-    <collision>
-      <origin xyz="0 0 0" rpy="0 0 0"/>
-      <geometry>
-    	<box size="0.005 0.006 0.0065"/>
-      </geometry>
-    </collision>
     <visual>
       <origin xyz="0 0 0" rpy="0 0 0"/>
@@ -574,13 +562,13 @@
         <scan>
           <horizontal>
-            <samples>200</samples>
+            <samples>100</samples>
             <resolution>1</resolution>
-            <min_angle>-1.5707963268</min_angle>
-            <max_angle>1.5707963268</max_angle>
+            <min_angle>-0.785398163</min_angle>
+            <max_angle>0.785398163</max_angle>
           </horizontal>
         </scan>
         <range>
           <min>0.0010</min>
-          <max>3.0</max>
+          <max>0.3</max>
           <resolution>0.01</resolution>
         </range>

Commit message: Cleaning camera project (not tested)

File: alphabot2_world/robots/alphabot2.xacro (robot description, xacro)
@@ -5,4 +5,5 @@
   <xacro:include filename="$(find alphabot2_world)/robots/wheel_macro.xacro" />
   <xacro:include filename="$(find alphabot2_world)/robots/caster_macro.xacro" />
+  <xacro:include filename="$(find alphabot2_world)/robots/pantilt.xacro" />
   <!-- chassis -->
   <link name="link_chassis">
@@ -50,5 +51,6 @@
   <!-- end of joint for left wheel -->
   <!-- Lower Camera-->
-  <link name="lower_camera_link">
+  <xacro:pan_tilt_link name="link_lower_camera" mass="0.0225" />
+  <!--<link name="link_lower_camera">
     <inertial>
       <mass value="0.0225"/>
@@ -69,21 +71,32 @@
       <material name="red"/>
     </visual>
-  </link>
-  <joint name="joint_lower_camera_link" type="continuous"><!--AQUI USAM REVOLUTE -->
+  </link>-->
+  <!-- joint pan -->
+  <xacro:pan_tilt_joint
+    name="joint_lower_camera"
+    type="continuous"
+    child="link_lower_camera"
+    parent="link_chassis"
+    origin_xyz="0 0 0.045">
+    <axis>
+      <axis rpy="0 0 0" xyz="0 0 1"/>
+    </axis>
+  </xacro:pan_tilt_joint>
+  <!-- end of joint pan -->
+  <!--<joint name="joint_link_lower_camera" type="continuous">
     <origin rpy="0 0 0" xyz="0 0 0.045"/>
-    <child link="lower_camera_link" />
+    <child link="link_lower_camera" />
     <parent link="link_chassis"/>
     <axis rpy="0 0 0" xyz="0 0 1"/>
     <limit effort="30" velocity="1" lower="-1.57" upper="1.57"/>
     <dynamics dampling="2" friction="2"/>
-  </joint>
-  <gazebo reference="lower_camera_link">
-        <material>Gazebo/Yellow</material>
-        <!--selfCollide>false</selfCollide>
-        <turnGravityOff>true</turnGravityOff-->
-  </gazebo>
-  <transmission name="pan_trans">
+  </joint>-->
+  <xacro:pan_tilt_transmission
+    name="pan"
+    joint="joint_lower_camera"
+  />
+  <!--<transmission name="pan_trans">
     <type>transmission_interface/SimpleTransmission</type>
-    <joint name="joint_lower_camera_link">
+    <joint name="joint_link_lower_camera">
       <hardwareInterface>PositionJointInterface</hardwareInterface>
     </joint>
@@ -91,8 +104,9 @@
       <mechanicalReduction>1</mechanicalReduction>
     </actuator>
-  </transmission>
+  </transmission>-->
   <!--End Lower Camera-->
   <!--Upper Camera-->
-  <link name="upper_camera_link">
+  <xacro:pan_tilt_link name="link_upper_camera" mass="0.0225" />
+  <!--<link name="link_upper_camera">
     <origin rpy="0 0 0" xyz="0 0 0"/>
     <inertial>
@@ -114,79 +128,25 @@
       <material name="blue"/>
     </visual>
-  </link>
-  <gazebo reference="upper_camera_link">
-        <material>Gazebo/Yellow</material>
-        <!--selfCollide>true</selfCollide>
-        <turnGravityOff>true</turnGravityOff-->
-  </gazebo>
-  <joint name="joint_upper_camera_link" type="revolute">
-    <origin rpy="0 0 0" xyz="0 0 0.045"/> <!--0.045-->
-    <child link="upper_camera_link" />
-    <parent link="lower_camera_link"/>
+  </link>-->
+  <xacro:pan_tilt_joint
+    name="joint_upper_camera"
+    type="revolute"
+    child="link_upper_camera"
+    parent="link_lower_camera"
+    origin_xyz="0 0 0.045">
+    <axis rpy="0 0 0" xyz="0 1 0 "/>
+  </xacro:pan_tilt_joint>
+  <!--<joint name="joint_link_upper_camera" type="revolute">
+    <origin rpy="0 0 0" xyz="0 0 0.045"/>
+    <child link="link_upper_camera" />
+    <parent link="link_lower_camera"/>
     <axis rpy="0 0 0" xyz="0 1 0"/>
     <limit effort="30" velocity="1" lower="-1.57" upper="1.57"/>
     <dynamics dampling="2" friction="2"/>
-  </joint>
-  <transmission name="tilt_trans">
-    <type>transmission_interface/SimpleTransmission</type>
-    <joint name="joint_upper_camera_link">
-      <hardwareInterface>PositionJointInterface</hardwareInterface>
-    </joint>
-    <actuator name="camera_tilt_motor">
-      <mechanicalReduction>1</mechanicalReduction>
-    </actuator>
-  </transmission>
+  </joint> -->
+  <xacro:pan_tilt_transmission
+    name="tilt"
+    joint="joint_upper_camera"
+  />
   <!--End Upper Camera-->
-  <!--For all the transmission tags; links gazebo with ROS-->
-  <gazebo>
-    <plugin name="gazebo_ros_control" filename="libgazebo_ros_control.so">
-      <robotNamespace>/alphabot2</robotNamespace>
-    </plugin>
-  </gazebo>
-  <!-- camera -->
-  <gazebo reference="upper_camera_link">
-    <sensor name="alphabot2_camera" type="camera" >
-      <visualize>1</visualize>
-      <always_on>1</always_on>
-      <update_rate>30.0</update_rate>
-      <camera name="alphabot2_camera">
-      <origin rpy="0 ${3.14/2} 0" xyz="0.015 0 0.045"/>
-        <save enabled="true">
-          <path>/tmp/</path>
-        </save>
-        <horizontal_fov>1.08504</horizontal_fov>
-        <image>
-          <width>160</width>
-          <height>120</height>
-          <format>R8G8B8</format>
-        </image>
-        <clip>
-          <near>0.01</near>
-          <far>1000</far>
-        </clip>
-        <noise>
-          <type>gaussian</type>
-          <!-- Noise is sampled independently per pixel on each frame.
-               That pixel's noise value is added to each of its color
-               channels, which at that point lie in the range [0,1]. -->
-          <mean>0.0</mean>
-          <stddev>0.007</stddev>
-        </noise>
-      </camera>
-      <plugin name="camera_controller" filename="libgazebo_ros_camera.so">
-        <alwaysOn>true</alwaysOn>
-        <updateRate>30.0</updateRate>
-        <cameraName>alphabot2_camera/</cameraName>
-        <imageTopicName>image_raw</imageTopicName>
-        <cameraInfoTopicName>camera_info</cameraInfoTopicName>
-        <frameName>camera_link</frameName>
-        <hackBaseline>0.07</hackBaseline>
-        <distortionK1>0.0</distortionK1>
-        <distortionK2>0.0</distortionK2>
-        <distortionK3>0.0</distortionK3>
-        <distortionT1>0.0</distortionT1>
-        <distortionT2>0.0</distortionT2>
-      </plugin>
-    </sensor>
-  </gazebo>
 </robot>

File: alphabot2_world/robots/gazebo.xacro (robot description, xacro)
@@ -11,6 +11,12 @@
     <material>Gazebo/Black</material>
   </gazebo>
-  <gazebo reference="upper_camera_link">
+  <gazebo reference="link_upper_camera">
     <material>Gazebo/Blue</material>
+  </gazebo>
+  <gazebo reference="link_lower_camera">
+    <material>Gazebo/Yellow</material>
+  </gazebo>
+  <gazebo reference="link_upper_camera">
+    <material>Gazebo/Yellow</material>
   </gazebo>
   <!-- end of gazebo colors definitions -->
@@ -31,4 +37,58 @@
     </plugin>
   </gazebo>
-  <!-- end of DIferential Control -->
+  <!-- end of Diferential Control -->
+  <!--For all the transmission tags; links gazebo with ROS-->
+  <gazebo>
+    <plugin name="gazebo_ros_control" filename="libgazebo_ros_control.so">
+      <robotNamespace>/alphabot2</robotNamespace>
+    </plugin>
+  </gazebo>
+  <!-- end of transmission tags-->
+  <!-- Camera -->
+  <gazebo reference="link_upper_camera">
+    <sensor name="alphabot2_camera" type="camera" >
+      <visualize>1</visualize>
+      <always_on>1</always_on>
+      <update_rate>30.0</update_rate>
+      <camera name="alphabot2_camera">
+      <origin rpy="0 ${3.14/2} 0" xyz="0.015 0 0.045"/>
+        <save enabled="true">
+          <path>/tmp/</path>
+        </save>
+        <horizontal_fov>1.08504</horizontal_fov>
+        <image>
+          <width>160</width>
+          <height>120</height>
+          <format>R8G8B8</format>
+        </image>
+        <clip>
+          <near>0.01</near>
+          <far>1000</far>
+        </clip>
+        <noise>
+          <type>gaussian</type>
+          <!-- Noise is sampled independently per pixel on each frame.
+               That pixel's noise value is added to each of its color
+               channels, which at that point lie in the range [0,1]. -->
+          <mean>0.0</mean>
+          <stddev>0.007</stddev>
+        </noise>
+      </camera>
+      <plugin name="camera_controller" filename="libgazebo_ros_camera.so">
+        <alwaysOn>true</alwaysOn>
+        <updateRate>30.0</updateRate>
+        <cameraName>alphabot2_camera/</cameraName>
+        <imageTopicName>image_raw</imageTopicName>
+        <cameraInfoTopicName>camera_info</cameraInfoTopicName>
+        <frameName>camera_link</frameName>
+        <hackBaseline>0.07</hackBaseline>
+        <distortionK1>0.0</distortionK1>
+        <distortionK2>0.0</distortionK2>
+        <distortionK3>0.0</distortionK3>
+        <distortionT1>0.0</distortionT1>
+        <distortionT2>0.0</distortionT2>
+      </plugin>
+    </sensor>
+  </gazebo>
+  <!-- end of Camera -->
 </robot>

Commit message: Fix Axis Xacro

File: alphabot2_world/robots/alphabot2.xacro (robot description, xacro)
@@ -78,9 +78,7 @@
     child="link_lower_camera"
     parent="link_chassis"
-    origin_xyz="0 0 0.045">
-    <axis>
-      <axis rpy="0 0 0" xyz="0 0 1"/>
-    </axis>
-  </xacro:pan_tilt_joint>
+    origin_xyz="0 0 0.045"
+    axis_xyz="0 0 1"
+    />
   <!-- end of joint pan -->
   <!--<joint name="joint_link_lower_camera" type="continuous">
@@ -134,7 +132,7 @@
     child="link_upper_camera"
     parent="link_lower_camera"
-    origin_xyz="0 0 0.045">
-    <axis rpy="0 0 0" xyz="0 1 0 "/>
-  </xacro:pan_tilt_joint>
+    origin_xyz="0 0 0.045"
+    axis="0 1 0"
+    />
   <!--<joint name="joint_link_upper_camera" type="revolute">
     <origin rpy="0 0 0" xyz="0 0 0.045"/>

File: alphabot2_world/robots/gazebo.xacro (robot description, xacro)
@@ -15,7 +15,4 @@
   </gazebo>
   <gazebo reference="link_lower_camera">
-    <material>Gazebo/Yellow</material>
-  </gazebo>
-  <gazebo reference="link_upper_camera">
     <material>Gazebo/Yellow</material>
   </gazebo>

File: alphabot2_world/robots/pantilt.xacro (robot description, xacro)
@@ -27,10 +27,10 @@
   <!-- end of pan tilt link -->
   <!-- pan tilt joint -->
-  <xacro:macro name="pan_tilt_joint" params="name type child parent origin_xyz **axis">
+  <xacro:macro name="pan_tilt_joint" params="name type child parent origin_xyz axis">
     <joint name="${name}" type="${type}">
       <origin rpy="0 0 0" xyz="${origin_xyz}"/>
       <child link="${child}"/>
       <parent link="${parent}"/>
-      <xacro:insert_block name="axis" />
+      <axis rpy="0 0 0" xyz="${axis_xyz}"/>
       <limit effort="30" velocity="1" lower="-1.57" upper="1.57"/>
       <dynamics dampling="2" friction="2"/>

Commit message: Fix Typo

File: alphabot2_world/robots/alphabot2.xacro (robot description, xacro)
@@ -133,5 +133,5 @@
     parent="link_lower_camera"
     origin_xyz="0 0 0.045"
-    axis="0 1 0"
+    axis_xyz="0 1 0"
     />
   <!--<joint name="joint_link_upper_camera" type="revolute">

File: alphabot2_world/robots/pantilt.xacro (robot description, xacro)
@@ -27,5 +27,5 @@
   <!-- end of pan tilt link -->
   <!-- pan tilt joint -->
-  <xacro:macro name="pan_tilt_joint" params="name type child parent origin_xyz axis">
+  <xacro:macro name="pan_tilt_joint" params="name type child parent origin_xyz axis_xyz">
     <joint name="${name}" type="${type}">
       <origin rpy="0 0 0" xyz="${origin_xyz}"/>

Commit message: Reverting to the state of the project before cleaning

File: alphabot2_world/robots/alphabot2.xacro (robot description, xacro)
@@ -5,5 +5,4 @@
   <xacro:include filename="$(find alphabot2_world)/robots/wheel_macro.xacro" />
   <xacro:include filename="$(find alphabot2_world)/robots/caster_macro.xacro" />
-  <xacro:include filename="$(find alphabot2_world)/robots/pantilt.xacro" />
   <!-- chassis -->
   <link name="link_chassis">
@@ -51,6 +50,5 @@
   <!-- end of joint for left wheel -->
   <!-- Lower Camera-->
-  <xacro:pan_tilt_link name="link_lower_camera" mass="0.0225" />
-  <!--<link name="link_lower_camera">
+  <link name="lower_camera_link">
     <inertial>
       <mass value="0.0225"/>
@@ -71,30 +69,21 @@
       <material name="red"/>
     </visual>
-  </link>-->
-  <!-- joint pan -->
-  <xacro:pan_tilt_joint
-    name="joint_lower_camera"
-    type="continuous"
-    child="link_lower_camera"
-    parent="link_chassis"
-    origin_xyz="0 0 0.045"
-    axis_xyz="0 0 1"
-    />
-  <!-- end of joint pan -->
-  <!--<joint name="joint_link_lower_camera" type="continuous">
+  </link>
+  <joint name="joint_lower_camera_link" type="continuous"><!--AQUI USAM REVOLUTE -->
     <origin rpy="0 0 0" xyz="0 0 0.045"/>
-    <child link="link_lower_camera" />
+    <child link="lower_camera_link" />
     <parent link="link_chassis"/>
     <axis rpy="0 0 0" xyz="0 0 1"/>
     <limit effort="30" velocity="1" lower="-1.57" upper="1.57"/>
     <dynamics dampling="2" friction="2"/>
-  </joint>-->
-  <xacro:pan_tilt_transmission
-    name="pan"
-    joint="joint_lower_camera"
-  />
-  <!--<transmission name="pan_trans">
+  </joint>
+  <gazebo reference="lower_camera_link">
+        <material>Gazebo/Yellow</material>
+        <!--selfCollide>false</selfCollide>
+        <turnGravityOff>true</turnGravityOff-->
+  </gazebo>
+  <transmission name="pan_trans">
     <type>transmission_interface/SimpleTransmission</type>
-    <joint name="joint_link_lower_camera">
+    <joint name="joint_lower_camera_link">
       <hardwareInterface>PositionJointInterface</hardwareInterface>
     </joint>
@@ -102,9 +91,8 @@
       <mechanicalReduction>1</mechanicalReduction>
     </actuator>
-  </transmission>-->
+  </transmission>
   <!--End Lower Camera-->
   <!--Upper Camera-->
-  <xacro:pan_tilt_link name="link_upper_camera" mass="0.0225" />
-  <!--<link name="link_upper_camera">
+  <link name="upper_camera_link">
     <origin rpy="0 0 0" xyz="0 0 0"/>
     <inertial>
@@ -126,25 +114,79 @@
       <material name="blue"/>
     </visual>
-  </link>-->
-  <xacro:pan_tilt_joint
-    name="joint_upper_camera"
-    type="revolute"
-    child="link_upper_camera"
-    parent="link_lower_camera"
-    origin_xyz="0 0 0.045"
-    axis_xyz="0 1 0"
-    />
-  <!--<joint name="joint_link_upper_camera" type="revolute">
-    <origin rpy="0 0 0" xyz="0 0 0.045"/>
-    <child link="link_upper_camera" />
-    <parent link="link_lower_camera"/>
+  </link>
+  <gazebo reference="upper_camera_link">
+        <material>Gazebo/Yellow</material>
+        <!--selfCollide>true</selfCollide>
+        <turnGravityOff>true</turnGravityOff-->
+  </gazebo>
+  <joint name="joint_upper_camera_link" type="revolute">
+    <origin rpy="0 0 0" xyz="0 0 0.045"/> <!--0.045-->
+    <child link="upper_camera_link" />
+    <parent link="lower_camera_link"/>
     <axis rpy="0 0 0" xyz="0 1 0"/>
     <limit effort="30" velocity="1" lower="-1.57" upper="1.57"/>
     <dynamics dampling="2" friction="2"/>
-  </joint> -->
-  <xacro:pan_tilt_transmission
-    name="tilt"
-    joint="joint_upper_camera"
-  />
+  </joint>
+  <transmission name="tilt_trans">
+    <type>transmission_interface/SimpleTransmission</type>
+    <joint name="joint_upper_camera_link">
+      <hardwareInterface>PositionJointInterface</hardwareInterface>
+    </joint>
+    <actuator name="camera_tilt_motor">
+      <mechanicalReduction>1</mechanicalReduction>
+    </actuator>
+  </transmission>
   <!--End Upper Camera-->
+  <!--For all the transmission tags; links gazebo with ROS-->
+  <gazebo>
+    <plugin name="gazebo_ros_control" filename="libgazebo_ros_control.so">
+      <robotNamespace>/alphabot2</robotNamespace>
+    </plugin>
+  </gazebo>
+  <!-- camera -->
+  <gazebo reference="upper_camera_link">
+    <sensor name="alphabot2_camera" type="camera" >
+      <visualize>1</visualize>
+      <always_on>1</always_on>
+      <update_rate>30.0</update_rate>
+      <camera name="alphabot2_camera">
+      <origin rpy="0 ${3.14/2} 0" xyz="0.015 0 0.045"/>
+        <save enabled="true">
+          <path>/tmp/</path>
+        </save>
+        <horizontal_fov>1.08504</horizontal_fov>
+        <image>
+          <width>160</width>
+          <height>120</height>
+          <format>R8G8B8</format>
+        </image>
+        <clip>
+          <near>0.01</near>
+          <far>1000</far>
+        </clip>
+        <noise>
+          <type>gaussian</type>
+          <!-- Noise is sampled independently per pixel on each frame.
+               That pixel's noise value is added to each of its color
+               channels, which at that point lie in the range [0,1]. -->
+          <mean>0.0</mean>
+          <stddev>0.007</stddev>
+        </noise>
+      </camera>
+      <plugin name="camera_controller" filename="libgazebo_ros_camera.so">
+        <alwaysOn>true</alwaysOn>
+        <updateRate>30.0</updateRate>
+        <cameraName>alphabot2_camera/</cameraName>
+        <imageTopicName>image_raw</imageTopicName>
+        <cameraInfoTopicName>camera_info</cameraInfoTopicName>
+        <frameName>camera_link</frameName>
+        <hackBaseline>0.07</hackBaseline>
+        <distortionK1>0.0</distortionK1>
+        <distortionK2>0.0</distortionK2>
+        <distortionK3>0.0</distortionK3>
+        <distortionT1>0.0</distortionT1>
+        <distortionT2>0.0</distortionT2>
+      </plugin>
+    </sensor>
+  </gazebo>
 </robot>

File: alphabot2_world/robots/gazebo.xacro (robot description, xacro)
@@ -11,9 +11,6 @@
     <material>Gazebo/Black</material>
   </gazebo>
-  <gazebo reference="link_upper_camera">
+  <gazebo reference="upper_camera_link">
     <material>Gazebo/Blue</material>
-  </gazebo>
-  <gazebo reference="link_lower_camera">
-    <material>Gazebo/Yellow</material>
   </gazebo>
   <!-- end of gazebo colors definitions -->
@@ -34,58 +31,4 @@
     </plugin>
   </gazebo>
-  <!-- end of Diferential Control -->
-  <!--For all the transmission tags; links gazebo with ROS-->
-  <gazebo>
-    <plugin name="gazebo_ros_control" filename="libgazebo_ros_control.so">
-      <robotNamespace>/alphabot2</robotNamespace>
-    </plugin>
-  </gazebo>
-  <!-- end of transmission tags-->
-  <!-- Camera -->
-  <gazebo reference="link_upper_camera">
-    <sensor name="alphabot2_camera" type="camera" >
-      <visualize>1</visualize>
-      <always_on>1</always_on>
-      <update_rate>30.0</update_rate>
-      <camera name="alphabot2_camera">
-      <origin rpy="0 ${3.14/2} 0" xyz="0.015 0 0.045"/>
-        <save enabled="true">
-          <path>/tmp/</path>
-        </save>
-        <horizontal_fov>1.08504</horizontal_fov>
-        <image>
-          <width>160</width>
-          <height>120</height>
-          <format>R8G8B8</format>
-        </image>
-        <clip>
-          <near>0.01</near>
-          <far>1000</far>
-        </clip>
-        <noise>
-          <type>gaussian</type>
-          <!-- Noise is sampled independently per pixel on each frame.
-               That pixel's noise value is added to each of its color
-               channels, which at that point lie in the range [0,1]. -->
-          <mean>0.0</mean>
-          <stddev>0.007</stddev>
-        </noise>
-      </camera>
-      <plugin name="camera_controller" filename="libgazebo_ros_camera.so">
-        <alwaysOn>true</alwaysOn>
-        <updateRate>30.0</updateRate>
-        <cameraName>alphabot2_camera/</cameraName>
-        <imageTopicName>image_raw</imageTopicName>
-        <cameraInfoTopicName>camera_info</cameraInfoTopicName>
-        <frameName>camera_link</frameName>
-        <hackBaseline>0.07</hackBaseline>
-        <distortionK1>0.0</distortionK1>
-        <distortionK2>0.0</distortionK2>
-        <distortionK3>0.0</distortionK3>
-        <distortionT1>0.0</distortionT1>
-        <distortionT2>0.0</distortionT2>
-      </plugin>
-    </sensor>
-  </gazebo>
-  <!-- end of Camera -->
+  <!-- end of DIferential Control -->
 </robot>
