Commit message: basic version of algorithm with sensors

File: alphabot2_world/robots/alphabot2.xacro (robot description, xacro)
@@ -487,5 +487,5 @@
   <joint name="sensor1_top_joint" type="fixed">
     <axis xyz="0 1 0" />
-    <origin xyz="0.0469 -0.022 -0.0183" rpy="0 0 0"/>
+    <origin xyz="0.0469 -0.022 -0.0183" rpy="0 0 -0.349066"/>
     <parent link="link_chassis"/>
     <child link="sensor1_top"/>
@@ -537,5 +537,5 @@
   <joint name="sensor2_top_joint" type="fixed">
     <axis xyz="0 1 0" />
-    <origin xyz="0.0469 0.022 -0.0183" rpy="0 0 0"/>
+    <origin xyz="0.0469 0.022 -0.0183" rpy="0 0 0.349066"/>
     <parent link="link_chassis"/>
     <child link="sensor2_top"/>

Commit message: Update alphabot2.xacro

File: alphabot2_world/robots/alphabot2.xacro (robot description, xacro)
@@ -24,5 +24,5 @@
       <origin rpy="0 0 0" xyz="0 0 -0.0065"/>
       <geometry>
-        <cylinder radius="0.055" length="0.045"/>
+        <mesh filename="package://alphabot2_world/meshes/chassis.stl" />
       </geometry>
       <material name="blue"/>
